Commit message: modified urdf to include lidar and gps

File: urdf/rover_sim.urdf.xacro (robot description, xacro)
@@ -193,9 +193,5 @@
   </link>
   <link name="imu_link"/>
-  <joint name="scan_joint" type="fixed">
-    <parent link="top_link"/>
-    <child link="lidar_link"/>
-    <origin xyz="0.125 0 0.05" rpy="0 0 0"/>
-  </joint>
+  <link name="gps_link"/>
   <link name="lidar_link">
     <visual>
@@ -221,4 +217,14 @@
   </link>
   <!-- Defining model joints. -->
+  <joint name="scan_joint" type="fixed">
+    <parent link="top_link"/>
+    <child link="lidar_link"/>
+    <origin xyz="0.125 0 0.05" rpy="0 0 0"/>
+  </joint>
+  <joint name="gps_joint" type="fixed">
+    <parent link="top_link"/>
+    <child link="gps_link"/>
+    <origin xyz="0.0 0 0.05" rpy="0 0 0"/>
+  </joint>
   <joint name="imu_joint" type="fixed">
     <parent link="base_link"/>

Commit message: [FIX] Removed incorrect odom transform

File: urdf/rover_sim.urdf.xacro (robot description, xacro)
@@ -91,5 +91,4 @@
   </xacro:macro>
   <!-- Defining model links. -->
-  <link name="odom" />
   <link
     name="base_link">
@@ -231,10 +230,4 @@
     <child link="imu_link"/>
     <origin xyz="0.0 0 0.068" rpy="0 0 0"/>
-  </joint>
-  <joint
-    name="fixed_base_joint"
-    type="fixed">
-    <parent link="odom" />
-    <child link="base_link" />
   </joint>
   <joint

Commit message: [FIX] missing odom link

File: urdf/rover_sim.urdf.xacro (robot description, xacro)
@@ -92,4 +92,7 @@
   <!-- Defining model links. -->
   <link
+    name="odom">
+  </link>
+  <link
     name="base_link">
     <inertial>

Commit message: [FIx] removed odom from urdf

File: urdf/rover_sim.urdf.xacro (robot description, xacro)
@@ -92,7 +92,4 @@
   <!-- Defining model links. -->
   <link
-    name="odom">
-  </link>
-  <link
     name="base_link">
     <inertial>

Commit message: [ADD] included camera_link

File: urdf/rover_sim.urdf.xacro (robot description, xacro)
@@ -115,5 +115,5 @@
     <collision>
       <origin
-        xyz="0 0 0.15"
+        xyz="0 0 0.12"
         rpy="0 0 0" />
       <geometry>
@@ -193,26 +193,6 @@
   <link name="imu_link"/>
   <link name="gps_link"/>
-  <link name="lidar_link">
-    <visual>
-      <origin xyz="0 0 0.0" rpy="0 0 0"/>
-      <geometry>
-        <mesh filename="package://rover_description/meshes/lds.stl" scale="0.001 0.001 0.001"/>
-      </geometry>
-      <material name="black"/>
-    </visual>
-    <collision>
-      <origin xyz="0.015 0 -0.0065" rpy="0 0 0"/>
-      <geometry>
-        <cylinder length="0.0315" radius="0.055"/>
-      </geometry>
-    </collision>
-    <inertial>
-      <mass value="0.114" />
-      <origin xyz="0 0 0" />
-      <inertia ixx="0.001" ixy="0.0" ixz="0.0"
-               iyy="0.001" iyz="0.0"
-               izz="0.001" />
-    </inertial>
-  </link>
+  <link name="lidar_link"/>
+  <link name="camera_link"/>
   <!-- Defining model joints. -->
   <joint name="scan_joint" type="fixed">
@@ -230,4 +210,9 @@
     <child link="imu_link"/>
     <origin xyz="0.0 0 0.068" rpy="0 0 0"/>
+  </joint>
+  <joint name="camera_joint" type="fixed">
+    <parent link="base_link"/>
+    <child link="camera_link"/>
+    <origin xyz="0.12 0 0.15" rpy="0 0 0"/>
   </joint>
   <joint

Commit message: [FIx] added optical frame link

File: urdf/rover_sim.urdf.xacro (robot description, xacro)
@@ -195,4 +195,5 @@
   <link name="lidar_link"/>
   <link name="camera_link"/>
+  <link name="camera_optical_link"/>
   <!-- Defining model joints. -->
   <joint name="scan_joint" type="fixed">
@@ -215,4 +216,9 @@
     <child link="camera_link"/>
     <origin xyz="0.12 0 0.15" rpy="0 0 0"/>
+  </joint>
+  <joint name="camera_optical_joint" type="fixed">
+    <origin xyz="0 0 0" rpy="${-pi/2} 0 ${-pi/2}"/>
+    <parent link="camera_link"/>
+    <child link="camera_optical_link"/>
   </joint>
   <joint

Commit message: [FIx] camera positioning

File: urdf/rover_sim.urdf.xacro (robot description, xacro)
@@ -95,5 +95,5 @@
     <inertial>
       <origin
-        xyz="-0.00019948 0 0.05685679"
+        xyz="-0.00019948 0 0.2"
         rpy="0 0 0" />
       <mass
@@ -195,5 +195,5 @@
   <link name="lidar_link"/>
   <link name="camera_link"/>
-  <link name="camera_optical_link"/>
+  <link name="camera_depth_optical_frame"/>
   <!-- Defining model joints. -->
   <joint name="scan_joint" type="fixed">
@@ -215,10 +215,10 @@
     <parent link="base_link"/>
     <child link="camera_link"/>
-    <origin xyz="0.12 0 0.15" rpy="0 0 0"/>
-  </joint>
-  <joint name="camera_optical_joint" type="fixed">
+    <origin xyz="0.12 0 0.2" rpy="0 0 0"/>
+  </joint>
+  <joint name="camera_depth_optical_joint" type="fixed">
     <origin xyz="0 0 0" rpy="${-pi/2} 0 ${-pi/2}"/>
     <parent link="camera_link"/>
-    <child link="camera_optical_link"/>
+    <child link="camera_depth_optical_frame"/>
   </joint>
   <joint

Commit message: [FIX] added joint state publisher

File: urdf/rover_sim.urdf.xacro (robot description, xacro)
@@ -95,8 +95,8 @@
     <inertial>
       <origin
-        xyz="-0.00019948 0 0.2"
-        rpy="0 0 0" />
-      <mass
-        value="5.0" />
+        xyz="-0.00019948 0 0.05685679"
+        rpy="0 0 0" />
+      <mass
+        value="3.12" />
       <inertia
         ixx="0.01468727"
@@ -200,5 +200,5 @@
     <parent link="top_link"/>
     <child link="lidar_link"/>
-    <origin xyz="0.125 0 0.05" rpy="0 0 0"/>
+    <origin xyz="0.0 0 0.15" rpy="0 0 0"/>
   </joint>
   <joint name="gps_joint" type="fixed">
@@ -215,5 +215,5 @@
     <parent link="base_link"/>
     <child link="camera_link"/>
-    <origin xyz="0.12 0 0.2" rpy="0 0 0"/>
+    <origin xyz="0.12 0 0.175" rpy="0 0 0"/>
   </joint>
   <joint name="camera_depth_optical_joint" type="fixed">

Commit message: [TEST] urdf

File: urdf/rover_sim.urdf.xacro (robot description, xacro)
@@ -26,5 +26,5 @@
 	<visual>
 	  <geometry>
-	    <mesh filename="package://rover_description/meshes/wheel_link.STL" />
+	    <mesh filename="file://rover_description/meshes/wheel_link.STL" />
 	  </geometry>
 	  <material name="black" />
@@ -32,5 +32,5 @@
       <collision>
         <geometry>
-          <mesh filename="package://rover_description/meshes/wheel_link_simple.STL" />
+          <mesh filename="file://rover_description/meshes/wheel_link_simple.STL" />
         </geometry>
       </collision>
@@ -71,5 +71,5 @@
       <visual>
         <geometry>
-          <mesh filename="package://rover_description/meshes/antenna_link.STL" />
+          <mesh filename="file://rover_description/meshes/antenna_link.STL" />
         </geometry>
         <material name="black" />
@@ -92,4 +92,7 @@
   <!-- Defining model links. -->
   <link
+    name="base_footprint">
+  </link>
+  <link
     name="base_link">
     <inertial>
@@ -109,5 +112,5 @@
     <visual>
       <geometry>
-        <mesh filename="package://rover_description/meshes/chassis_link.STL" />
+        <mesh filename="file://rover_description/meshes/chassis_link.STL" />
       </geometry>
       <material name="gray" />
@@ -140,5 +143,5 @@
     <visual>
       <geometry>
-        <mesh filename="package://rover_description/meshes/top_link.STL" />
+        <mesh filename="file://rover_description/meshes/top_link.STL" />
       </geometry>
       <material name="white" />
@@ -163,5 +166,5 @@
     <visual>
       <geometry>
-        <mesh filename="package://rover_description/meshes/battery_link.STL" />
+        <mesh filename="file://rover_description/meshes/battery_link.STL" />
       </geometry>
       <material name="black" />
@@ -186,5 +189,5 @@
     <visual>
       <geometry>
-        <mesh filename="package://rover_description/meshes/housing_link.STL" />
+        <mesh filename="file://rover_description/meshes/housing_link.STL" />
       </geometry>
       <material name="black" />
@@ -197,4 +200,9 @@
   <link name="camera_depth_optical_frame"/>
   <!-- Defining model joints. -->
+  <joint name="base_joint" type="fixed">
+    <parent link="base_footprint"/>
+    <child link="base_link"/>
+    <origin xyz="0.0 0 0.1" rpy="0 0 0"/>
+  </joint>
   <joint name="scan_joint" type="fixed">
     <parent link="top_link"/>

Commit message: [FIX] incorrect file path

File: urdf/rover_sim.urdf.xacro (robot description, xacro)
@@ -26,5 +26,5 @@
 	<visual>
 	  <geometry>
-	    <mesh filename="file://rover_description/meshes/wheel_link.STL" />
+	    <mesh filename="file://$(env HOME)/rover_description/meshes/wheel_link.STL" />
 	  </geometry>
 	  <material name="black" />
@@ -32,5 +32,5 @@
       <collision>
         <geometry>
-          <mesh filename="file://rover_description/meshes/wheel_link_simple.STL" />
+          <mesh filename="file://$(env HOME)/rover_description/meshes/wheel_link_simple.STL" />
         </geometry>
       </collision>
@@ -71,5 +71,5 @@
       <visual>
         <geometry>
-          <mesh filename="file://rover_description/meshes/antenna_link.STL" />
+          <mesh filename="file://$(env HOME)/rover_description/meshes/antenna_link.STL" />
         </geometry>
         <material name="black" />
@@ -112,5 +112,5 @@
     <visual>
       <geometry>
-        <mesh filename="file://rover_description/meshes/chassis_link.STL" />
+        <mesh filename="file://$(env HOME)/rover_description/meshes/chassis_link.STL" />
       </geometry>
       <material name="gray" />
@@ -143,5 +143,5 @@
     <visual>
       <geometry>
-        <mesh filename="file://rover_description/meshes/top_link.STL" />
+        <mesh filename="file://$(env HOME)/rover_description/meshes/top_link.STL" />
       </geometry>
       <material name="white" />
@@ -166,5 +166,5 @@
     <visual>
       <geometry>
-        <mesh filename="file://rover_description/meshes/battery_link.STL" />
+        <mesh filename="file://$(env HOME)/rover_description/meshes/battery_link.STL" />
       </geometry>
       <material name="black" />
@@ -189,5 +189,5 @@
     <visual>
       <geometry>
-        <mesh filename="file://rover_description/meshes/housing_link.STL" />
+        <mesh filename="file://$(env HOME)/rover_description/meshes/housing_link.STL" />
       </geometry>
       <material name="black" />

Commit message: [FIX] path

File: urdf/rover_sim.urdf.xacro (robot description, xacro)
@@ -26,5 +26,5 @@
 	<visual>
 	  <geometry>
-	    <mesh filename="file://$(env HOME)/rover_description/meshes/wheel_link.STL" />
+	    <mesh filename="file://$(env HOME)/rover/src/rover_description/meshes/wheel_link.STL" />
 	  </geometry>
 	  <material name="black" />
@@ -32,5 +32,5 @@
       <collision>
         <geometry>
-          <mesh filename="file://$(env HOME)/rover_description/meshes/wheel_link_simple.STL" />
+          <mesh filename="file://$(env HOME)/rover/src/rover_description/meshes/wheel_link_simple.STL" />
         </geometry>
       </collision>
@@ -71,5 +71,5 @@
       <visual>
         <geometry>
-          <mesh filename="file://$(env HOME)/rover_description/meshes/antenna_link.STL" />
+          <mesh filename="file://$(env HOME)/rover/src/rover_description/meshes/antenna_link.STL" />
         </geometry>
         <material name="black" />
@@ -112,5 +112,5 @@
     <visual>
       <geometry>
-        <mesh filename="file://$(env HOME)/rover_description/meshes/chassis_link.STL" />
+        <mesh filename="file://$(env HOME)/rover/src/rover_description/meshes/chassis_link.STL" />
       </geometry>
       <material name="gray" />
@@ -143,5 +143,5 @@
     <visual>
       <geometry>
-        <mesh filename="file://$(env HOME)/rover_description/meshes/top_link.STL" />
+        <mesh filename="file://$(env HOME)/rover/src/rover_description/meshes/top_link.STL" />
       </geometry>
       <material name="white" />
@@ -166,5 +166,5 @@
     <visual>
       <geometry>
-        <mesh filename="file://$(env HOME)/rover_description/meshes/battery_link.STL" />
+        <mesh filename="file://$(env HOME)/rover/src/rover_description/meshes/battery_link.STL" />
       </geometry>
       <material name="black" />
@@ -189,5 +189,5 @@
     <visual>
       <geometry>
-        <mesh filename="file://$(env HOME)/rover_description/meshes/housing_link.STL" />
+        <mesh filename="file://$(env HOME)/rover/src/rover_description/meshes/housing_link.STL" />
       </geometry>
       <material name="black" />

Commit message: [FIX] reverted to package call

File: urdf/rover_sim.urdf.xacro (robot description, xacro)
@@ -26,5 +26,5 @@
 	<visual>
 	  <geometry>
-	    <mesh filename="file://$(env HOME)/rover/src/rover_description/meshes/wheel_link.STL" />
+	    <mesh filename="package://rover_description/meshes/wheel_link.STL" />
 	  </geometry>
 	  <material name="black" />
@@ -32,5 +32,5 @@
       <collision>
         <geometry>
-          <mesh filename="file://$(env HOME)/rover/src/rover_description/meshes/wheel_link_simple.STL" />
+          <mesh filename="package://rover_description/meshes/wheel_link_simple.STL" />
         </geometry>
       </collision>
@@ -71,5 +71,5 @@
       <visual>
         <geometry>
-          <mesh filename="file://$(env HOME)/rover/src/rover_description/meshes/antenna_link.STL" />
+          <mesh filename="package://rover_description/meshes/antenna_link.STL" />
         </geometry>
         <material name="black" />
@@ -112,5 +112,5 @@
     <visual>
       <geometry>
-        <mesh filename="file://$(env HOME)/rover/src/rover_description/meshes/chassis_link.STL" />
+        <mesh filename="package://rover_description/meshes/chassis_link.STL" />
       </geometry>
       <material name="gray" />
@@ -143,5 +143,5 @@
     <visual>
       <geometry>
-        <mesh filename="file://$(env HOME)/rover/src/rover_description/meshes/top_link.STL" />
+        <mesh filename="package://rover_description/meshes/top_link.STL" />
       </geometry>
       <material name="white" />
@@ -166,5 +166,5 @@
     <visual>
       <geometry>
-        <mesh filename="file://$(env HOME)/rover/src/rover_description/meshes/battery_link.STL" />
+        <mesh filename="package://rover_description/meshes/battery_link.STL" />
       </geometry>
       <material name="black" />
@@ -189,5 +189,5 @@
     <visual>
       <geometry>
-        <mesh filename="file://$(env HOME)/rover/src/rover_description/meshes/housing_link.STL" />
+        <mesh filename="package://rover_description/meshes/housing_link.STL" />
       </geometry>
       <material name="black" />

Commit message: [TEST]

File: urdf/rover_sim.urdf.xacro (robot description, xacro)
@@ -26,5 +26,5 @@
 	<visual>
 	  <geometry>
-	    <mesh filename="package://rover_description/meshes/wheel_link.STL" />
+	    <mesh filename="package://$(find rover_description)/meshes/wheel_link.STL" />
 	  </geometry>
 	  <material name="black" />
@@ -32,5 +32,5 @@
       <collision>
         <geometry>
-          <mesh filename="package://rover_description/meshes/wheel_link_simple.STL" />
+          <mesh filename="package://$(find rover_description)/meshes/wheel_link_simple.STL" />
         </geometry>
       </collision>
@@ -71,5 +71,5 @@
       <visual>
         <geometry>
-          <mesh filename="package://rover_description/meshes/antenna_link.STL" />
+          <mesh filename="package://$(find rover_description)/meshes/antenna_link.STL" />
         </geometry>
         <material name="black" />
@@ -112,5 +112,5 @@
     <visual>
       <geometry>
-        <mesh filename="package://rover_description/meshes/chassis_link.STL" />
+        <mesh filename="package://$(find rover_description)/meshes/chassis_link.STL" />
       </geometry>
       <material name="gray" />
@@ -143,5 +143,5 @@
     <visual>
       <geometry>
-        <mesh filename="package://rover_description/meshes/top_link.STL" />
+        <mesh filename="package://$(find rover_description)/meshes/top_link.STL" />
       </geometry>
       <material name="white" />
@@ -166,5 +166,5 @@
     <visual>
       <geometry>
-        <mesh filename="package://rover_description/meshes/battery_link.STL" />
+        <mesh filename="package://$(find rover_description)/meshes/battery_link.STL" />
       </geometry>
       <material name="black" />
@@ -189,5 +189,5 @@
     <visual>
       <geometry>
-        <mesh filename="package://rover_description/meshes/housing_link.STL" />
+        <mesh filename="package://$(find rover_description)/meshes/housing_link.STL" />
       </geometry>
       <material name="black" />

Commit message: [FIX] mesh file path

File: urdf/rover_sim.urdf.xacro (robot description, xacro)
@@ -26,5 +26,5 @@
 	<visual>
 	  <geometry>
-	    <mesh filename="package://$(find rover_description)/meshes/wheel_link.STL" />
+	    <mesh filename="file://$(find rover_description)/meshes/wheel_link.STL" />
 	  </geometry>
 	  <material name="black" />
@@ -32,5 +32,5 @@
       <collision>
         <geometry>
-          <mesh filename="package://$(find rover_description)/meshes/wheel_link_simple.STL" />
+          <mesh filename="file://$(find rover_description)/meshes/wheel_link_simple.STL" />
         </geometry>
       </collision>
@@ -71,5 +71,5 @@
       <visual>
         <geometry>
-          <mesh filename="package://$(find rover_description)/meshes/antenna_link.STL" />
+          <mesh filename="file://$(find rover_description)/meshes/antenna_link.STL" />
         </geometry>
         <material name="black" />
@@ -112,5 +112,5 @@
     <visual>
       <geometry>
-        <mesh filename="package://$(find rover_description)/meshes/chassis_link.STL" />
+        <mesh filename="file://$(find rover_description)/meshes/chassis_link.STL" />
       </geometry>
       <material name="gray" />
@@ -143,5 +143,5 @@
     <visual>
       <geometry>
-        <mesh filename="package://$(find rover_description)/meshes/top_link.STL" />
+        <mesh filename="file://$(find rover_description)/meshes/top_link.STL" />
       </geometry>
       <material name="white" />
@@ -166,5 +166,5 @@
     <visual>
       <geometry>
-        <mesh filename="package://$(find rover_description)/meshes/battery_link.STL" />
+        <mesh filename="file://$(find rover_description)/meshes/battery_link.STL" />
       </geometry>
       <material name="black" />
@@ -189,5 +189,5 @@
     <visual>
       <geometry>
-        <mesh filename="package://$(find rover_description)/meshes/housing_link.STL" />
+        <mesh filename="file://$(find rover_description)/meshes/housing_link.STL" />
       </geometry>
       <material name="black" />

Commit message: [FIx] removed link

File: urdf/rover_sim.urdf.xacro (robot description, xacro)
@@ -91,7 +91,7 @@
   </xacro:macro>
   <!-- Defining model links. -->
-  <link
+  <!-- <link
     name="base_footprint">
-  </link>
+  </link> -->
   <link
     name="base_link">
@@ -200,9 +200,9 @@
   <link name="camera_depth_optical_frame"/>
   <!-- Defining model joints. -->
-  <joint name="base_joint" type="fixed">
+  <!-- <joint name="base_joint" type="fixed">
     <parent link="base_footprint"/>
     <child link="base_link"/>
     <origin xyz="0.0 0 0.1" rpy="0 0 0"/>
-  </joint>
+  </joint> -->
   <joint name="scan_joint" type="fixed">
     <parent link="top_link"/>
